File: board/Main.sch (EAGLE design)
At the start: 31 parts, among them IC1 LP2950Z, J2 MICRO-SD_CARD_SOCKET, Q1 16MHz, U1 ATMEGA328P-PU

Commit message: Update Note 1 in schematic
Other:
- note added: "1. Solder these pads together to cause the controller to reset when the computer resets (Manual resets are still possible, but they will not reset the computer). Leave open for manual reset only."
- note removed: "1. Solder these pads together to cause the controler to reset when the computer resets (Manual resets are still possible, but they will not reset the computer). Leave open for manual reset only."
Changed lines of the file:
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@@
 <text x="124.714" y="56.642" size="1.778" layer="97">See Note 1</text>
 <text x="203.2" y="129.54" size="1.778" layer="97">1. Solder these pads together to cause
-the controler to reset when the computer
+the controller to reset when the computer
 resets (Manual resets are still possible,
 but they will not reset the computer).
